File: tz1-mvb/tz1-mvb.kicad_pcb (KiCad board)
At the start: 2 copper layers, 12 parts, among them J1 Conn_01x03, J2 AudioJack2_Ground, Q1 BC547, Q2 BC547

Commit message: Finally found my parts
Parts:
- removed J2: AudioJack2_Ground, Connector_Audio:Jack_3.5mm_CUI_SJ-3523-SMT_Horizontal
- moved C2 1437.1 mm to (70.9, -26.7)
- moved J1 1437.1 mm to (31.4, -31.2)
- moved Q2 1437.1 mm to (77.3, -43.5)
- moved R3 1437.1 mm to (44.0, -26.0)
- moved R4 1437.1 mm to (57.4, -26.0)
- moved C1 1437.1 mm to (70.9, -30.3)
- moved C3 1437.1 mm to (70.9, -23.2)
- moved Q1 1437.1 mm to (77.9, -47.8)
- moved R1 1437.1 mm to (44.0, -30.0)
- moved R2 1437.1 mm to (57.4, -30.0)
- moved RV1 1437.1 mm to (31.3, -37.3)
Other:
- board text added: "TEST"

Commit message: Manually rendered
Parts:
- moved Q1 105.2 mm to (-25.4, -27.4), turned to 270 degrees
- moved C1 87.9 mm to (-17.0, -31.5), turned to 180 degrees
- moved Q2 83.3 mm to (-3.81, -24.1), turned to 90 degrees
- moved R2 77.3 mm to (-17.8, -48.3), turned to 270 degrees
- moved C2 71.2 mm to (-0.08, -33.0), turned to 180 degrees
- moved R1 71.2 mm to (-25.4, -45.7), turned to 270 degrees
- moved C3 71.2 mm to (2.54, -43.2), turned to 270 degrees
- moved R4 63.9 mm to (-2.54, -48.3), turned to 270 degrees
- moved R3 58.0 mm to (-10.2, -46.5), turned to 270 degrees
- moved J1 29.2 mm to (7.62, -48.3)
- moved RV1 26.5 mm to (7.62, -25.6)
Routing:
- net GND: track 0.00 -> 55.1 mm
- net VCC: track 0.00 -> 35.5 mm
- net Net-(C2-Pad1): track 0.00 -> 31.1 mm
- net Net-(C2-Pad2): track 0.00 -> 28.1 mm
- net Net-(C1-Pad1): track 0.00 -> 22.4 mm
- net Net-(C3-Pad2): track 0.00 -> 11.2 mm
- net Net-(C1-Pad2): track 0.00 -> 10.9 mm
- net /WAVE_OUT: track 0.00 -> 6.13 mm
Other:
- board outline added: 48 x 31 mm
- board text added: "PCB Rev 1.0"
- board text removed: "TEST"
