File: tz1-mvb/tz1-mvb.kicad_pcb (KiCad board)
At the start: 2 copper layers, 48 x 31 mm, 11 parts, among them J1 Conn_01x03, Q1 BC547, Q2 BC547

Commit message: Fixed board frame (DRC reported non-closed polygon)
Other:
- board size 48 x 31 mm -> 49.5 x 33 mm
Changed lines of the file:
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@@
   (general
     (thickness 1.6)
-    (drawings 7)
+    (drawings 6)
     (tracks 46)
     (zones 0)
@@
     )
   )
+  (dimension 49.53 (width 0.15) (layer Dwgs.User)
+    (gr_text "49.530 mm" (at -6.985 -11.4) (layer Dwgs.User)
+      (effects (font (size 1 1) (thickness 0.15)))
+    )
+    (feature1 (pts (xy 17.78 -15.24) (xy 17.78 -12.113579)))
+    (feature2 (pts (xy -31.75 -15.24) (xy -31.75 -12.113579)))
+    (crossbar (pts (xy -31.75 -12.7) (xy 17.78 -12.7)))
+    (arrow1a (pts (xy 17.78 -12.7) (xy 16.653496 -12.113579)))
+    (arrow1b (pts (xy 17.78 -12.7) (xy 16.653496 -13.286421)))
+    (arrow2a (pts (xy -31.75 -12.7) (xy -30.623496 -12.113579)))
+    (arrow2b (pts (xy -31.75 -12.7) (xy -30.623496 -13.286421)))
+  )
+  (gr_line (start -31.75 -19.05) (end 17.78 -19.05) (layer Edge.Cuts) (width 0.05))
+  (gr_line (start -31.75 -52.07) (end -31.75 -19.05) (layer Edge.Cuts) (width 0.05))
+  (gr_line (start 17.78 -52.07) (end -31.75 -52.07) (layer Edge.Cuts) (width 0.05))
+  (gr_line (start 17.78 -19.05) (end 17.78 -52.07) (layer Edge.Cuts) (width 0.05))
   (gr_text "PCB Rev 1.0" (at 15.24 -43.18 90) (layer B.Cu)
     (effects (font (size 1.5 1.5) (thickness 0.3)) (justify mirror))
   )
-  (dimension 48.26 (width 0.15) (layer Dwgs.User)
-    (gr_text "48.260 mm" (at -6.35 -13.94) (layer Dwgs.User)
-      (effects (font (size 1 1) (thickness 0.15)))
-    )
-    (feature1 (pts (xy 17.78 -17.78) (xy 17.78 -14.653579)))
-    (feature2 (pts (xy -30.48 -17.78) (xy -30.48 -14.653579)))
-    (crossbar (pts (xy -30.48 -15.24) (xy 17.78 -15.24)))
-    (arrow1a (pts (xy 17.78 -15.24) (xy 16.653496 -14.653579)))
-    (arrow1b (pts (xy 17.78 -15.24) (xy 16.653496 -15.826421)))
-    (arrow2a (pts (xy -30.48 -15.24) (xy -29.353496 -14.653579)))
-    (arrow2b (pts (xy -30.48 -15.24) (xy -29.353496 -15.826421)))
-  )
-  (gr_line (start -30.226 -20.066) (end -22.352 -20.066) (layer Edge.Cuts) (width 0.05))
-  (gr_line (start -30.226 -51.054) (end -30.226 -20.066) (layer Edge.Cuts) (width 0.05))
-  (gr_line (start 17.78 -51.054) (end -30.226 -51.054) (layer Edge.Cuts) (width 0.05))
-  (gr_line (start 17.78 -20.066) (end 17.78 -51.054) (layer Edge.Cuts) (width 0.05))
-  (gr_line (start -22.606 -20.066) (end 17.78 -20.066) (layer Edge.Cuts) (width 0.05))
   (segment (start -17.78 -32.258) (end -17.018 -31.496) (width 1.27) (layer F.Cu) (net 1))
   (segment (start -17.78 -38.1) (end -17.78 -32.258) (width 1.27) (layer F.Cu) (net 1))

Commit message: Forgotten change
Routing:
- net Net-(C2-Pad1): track 31.1 -> 26.5 mm
- net Net-(C2-Pad2): track 28.1 -> 25.2 mm
- net Net-(C1-Pad2): track 10.9 -> 11.7 mm
Changed lines of the file:
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@@
     (thickness 1.6)
     (drawings 6)
-    (tracks 46)
+    (tracks 43)
     (zones 0)
     (modules 11)
@@
   (segment (start -12.7 -25.4) (end -17.018 -29.718) (width 1.27) (layer B.Cu) (net 1))
   (segment (start -5.08 -25.4) (end -12.7 -25.4) (width 1.27) (layer B.Cu) (net 1))
-  (segment (start -25.4 -34.878) (end -22.018 -31.496) (width 1.27) (layer F.Cu) (net 2))
-  (segment (start -25.4 -35.56) (end -25.4 -34.878) (width 1.27) (layer F.Cu) (net 2))
-  (segment (start -25.4 -28.114) (end -22.018 -31.496) (width 1.27) (layer F.Cu) (net 2))
-  (segment (start -25.4 -27.432) (end -25.4 -28.114) (width 1.27) (layer F.Cu) (net 2))
-  (segment (start -6.858 -33.02) (end -10.16 -36.322) (width 1.27) (layer F.Cu) (net 3))
-  (segment (start -5.08 -33.02) (end -6.858 -33.02) (width 1.27) (layer F.Cu) (net 3))
-  (segment (start -24.13 -25.819802) (end -23.710198 -25.4) (width 1.27) (layer F.Cu) (net 3))
-  (segment (start -24.13 -26.162) (end -24.13 -25.819802) (width 1.27) (layer F.Cu) (net 3))
-  (segment (start -23.710198 -25.4) (end -16.51 -25.4) (width 1.27) (layer F.Cu) (net 3))
-  (segment (start -10.16 -31.75) (end -10.16 -36.322) (width 1.27) (layer F.Cu) (net 3))
-  (segment (start -16.51 -25.4) (end -10.16 -31.75) (width 1.27) (layer F.Cu) (net 3))
+  (segment (start -25.019 -31.496) (end -25.4 -31.115) (width 1.27) (layer F.Cu) (net 2))
+  (segment (start -22.018 -31.496) (end -25.019 -31.496) (width 1.27) (layer F.Cu) (net 2))
+  (segment (start -25.4 -31.115) (end -25.4 -35.56) (width 1.27) (layer F.Cu) (net 2))
+  (segment (start -25.4 -27.432) (end -25.4 -31.115) (width 1.27) (layer F.Cu) (net 2))
+  (segment (start -5.08 -33.02) (end -10.16 -33.02) (width 1.27) (layer F.Cu) (net 3))
+  (segment (start -10.16 -33.02) (end -10.16 -36.322) (width 1.27) (layer F.Cu) (net 3))
+  (segment (start -17.018 -26.162) (end -10.16 -33.02) (width 1.27) (layer F.Cu) (net 3))
+  (segment (start -24.13 -26.162) (end -17.018 -26.162) (width 1.27) (layer F.Cu) (net 3))
   (segment (start -2.54 -35.48) (end -0.08 -33.02) (width 1.27) (layer F.Cu) (net 4))
   (segment (start -2.54 -38.1) (end -2.54 -35.48) (width 1.27) (layer F.Cu) (net 4))
-  (segment (start 7.62 -25.56) (end 4.92 -25.56) (width 1.27) (layer F.Cu) (net 4))
-  (segment (start -0.08 -30.56) (end -0.08 -33.02) (width 1.27) (layer F.Cu) (net 4))
-  (segment (start 4.92 -25.56) (end -0.08 -30.56) (width 1.27) (layer F.Cu) (net 4))
   (segment (start -3.81 -24.13) (end 0 -24.13) (width 1.27) (layer F.Cu) (net 4))
   (segment (start 0 -32.94) (end -0.08 -33.02) (width 1.27) (layer F.Cu) (net 4))
-  (segment (start 0 -24.13) (end 0 -32.94) (width 1.27) (layer F.Cu) (net 4))
+  (segment (start 7.62 -25.56) (end 0.16 -25.56) (width 1.27) (layer F.Cu) (net 4))
+  (segment (start 0 -25.4) (end 0 -32.94) (width 1.27) (layer F.Cu) (net 4))
+  (segment (start 0.16 -25.56) (end 0 -25.4) (width 1.27) (layer F.Cu) (net 4))
+  (segment (start 0 -24.13) (end 0 -25.4) (width 1.27) (layer F.Cu) (net 4))
   (segment (start 5.08 -45.72) (end 2.54 -43.18) (width 1.27) (layer F.Cu) (net 5))
   (segment (start 7.62 -45.72) (end 5.08 -45.72) (width 1.27) (layer F.Cu) (net 5))
